File: veh_wirings/veh_wiring.sch (EAGLE design)
At the start: 0 parts

Commit message: 020120: TCU implemented and given to Lauri Lassila
Other:
- note added: "4200mm"
- note added: "4300mm"
- note added: "550mm"
- note added: "600mm"
- note added: "650mm"
- note added: "CM loading space"
- note removed: "4500 mm"
Changed lines of the file:
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@@
 <part name="U$8" library="uw_wiring_harness" deviceset="PIN" device="" value="1/3"/>
 <part name="U$9" library="uw_wiring_harness" deviceset="PIN" device="" value="2/3"/>
+<part name="U$10" library="uw_wiring_harness (usevolt-ThinkPad-X250's conflicted copy 2018-02-07)" deviceset="DT04-4P" device=""/>
+<part name="1/4" library="uw_wiring_harness (usevolt-ThinkPad-X250's conflicted copy 2018-02-07)" deviceset="PIN" device="" value="1/4"/>
+<part name="1/1" library="uw_wiring_harness (usevolt-ThinkPad-X250's conflicted copy 2018-02-07)" deviceset="PIN" device="" value="2/4"/>
+<part name="1/2" library="uw_wiring_harness (usevolt-ThinkPad-X250's conflicted copy 2018-02-07)" deviceset="PIN" device="" value="3/4"/>
+<part name="1/3" library="uw_wiring_harness (usevolt-ThinkPad-X250's conflicted copy 2018-02-07)" deviceset="PIN" device="" value="4/4"/>
+<part name="FRAME1" library="frames" deviceset="A3L-LOC" device=""/>
+<part name="U$22" library="uw_wiring_harness (usevolt-ThinkPad-X250's conflicted copy 2018-02-07)" deviceset="DT04-4P" device=""/>
+<part name="1/5" library="uw_wiring_harness (usevolt-ThinkPad-X250's conflicted copy 2018-02-07)" deviceset="PIN" device="" value="1/4"/>
+<part name="1/6" library="uw_wiring_harness (usevolt-ThinkPad-X250's conflicted copy 2018-02-07)" deviceset="PIN" device="" value="2/4"/>
+<part name="1/7" library="uw_wiring_harness (usevolt-ThinkPad-X250's conflicted copy 2018-02-07)" deviceset="PIN" device="" value="3/4"/>
+<part name="1/8" library="uw_wiring_harness (usevolt-ThinkPad-X250's conflicted copy 2018-02-07)" deviceset="PIN" device="" value="4/4"/>
+<part name="1/9" library="uw_wiring_harness (usevolt-ThinkPad-X250's conflicted copy 2018-02-07)" deviceset="PIN" device="" value="1/4"/>
+<part name="1/10" library="uw_wiring_harness (usevolt-ThinkPad-X250's conflicted copy 2018-02-07)" deviceset="PIN" device="" value="2/4"/>
+<part name="1/11" library="uw_wiring_harness (usevolt-ThinkPad-X250's conflicted copy 2018-02-07)" deviceset="PIN" device="" value="3/4"/>
+<part name="1/12" library="uw_wiring_harness (usevolt-ThinkPad-X250's conflicted copy 2018-02-07)" deviceset="PIN" device="" value="4/4"/>
+<part name="1/13" library="uw_wiring_harness (usevolt-ThinkPad-X250's conflicted copy 2018-02-07)" deviceset="DT06-4S" device=""/>
 </parts>
 <sheets>
@@
 <dimension x1="170.18" y1="190.5" x2="144.78" y2="190.5" x3="170.18" y3="190.5" textsize="5.08" textratio="10" layer="103" dtype="leader" width="0.254"/>
 <dimension x1="129.54" y1="190.5" x2="144.78" y2="190.5" x3="170.18" y3="190.5" textsize="2.54" layer="103" dtype="leader" width="0.254"/>
-<text x="143.256" y="192.024" size="2.54" layer="103" font="vector">4500 mm</text>
+<text x="143.256" y="192.024" size="2.54" layer="103" font="vector">4200mm</text>
 <text x="141.478" y="181.102" size="2.54" layer="101" font="vector">1.50mm2</text>
 <text x="141.478" y="186.182" size="2.54" layer="100" font="vector">1.50mm2</text>
@@
 <instance part="U$45" gate="G$1" x="58.42" y="198.12" rot="MR0"/>
 <instance part="U$262" gate="PIN" x="71.12" y="198.12"/>
+<instance part="U$10" gate="G$1" x="228.6" y="175.26"/>
+<instance part="1/4" gate="PIN" x="187.96" y="185.42" rot="MR0"/>
+<instance part="1/1" gate="PIN" x="187.96" y="180.34" rot="MR0"/>
+<instance part="1/2" gate="PIN" x="187.96" y="170.18" rot="MR0"/>
+<instance part="1/3" gate="PIN" x="187.96" y="165.1" rot="MR0"/>
+</instances>
+<busses>
+</busses>
+<nets>
+</nets>
+</sheet>
+<sheet>
+<plain>
+<text x="289.56" y="10.16" size="2.1844" layer="94" font="vector">Trailer Wirings
+Usewood Trailer
+(c) Usewood Forest Tec Oy
+Author: Olli Usenius</text>
+<text x="342.9" y="20.32" size="2.54" layer="94" font="vector">CM loading space</text>
+<wire x1="187.96" y1="185.42" x2="99.06" y2="185.42" width="0.254" layer="100"/>
+<wire x1="187.96" y1="180.34" x2="99.06" y2="180.34" width="0.254" layer="101"/>
+<wire x1="170.18" y1="190.5" x2="170.18" y2="162.56" width="0.254" layer="103" style="longdash"/>
+<wire x1="129.54" y1="190.5" x2="129.54" y2="162.56" width="0.254" layer="103" style="longdash"/>
+<dimension x1="170.18" y1="190.5" x2="144.78" y2="190.5" x3="170.18" y3="190.5" textsize="5.08" textratio="10" layer="103" dtype="leader" width="0.254"/>
+<dimension x1="129.54" y1="190.5" x2="144.78" y2="190.5" x3="170.18" y3="190.5" textsize="2.54" layer="103" dtype="leader" width="0.254"/>
+<text x="143.256" y="192.024" size="2.54" layer="103" font="vector">4300mm</text>
+<text x="141.478" y="181.102" size="2.54" layer="101" font="vector">1.50mm2</text>
+<text x="141.478" y="186.182" size="2.54" layer="100" font="vector">1.50mm2</text>
+<wire x1="132.08" y1="165.1" x2="132.08" y2="185.42" width="0.254" layer="103"/>
+<wire x1="132.08" y1="185.42" x2="137.16" y2="185.42" width="0.254" layer="103" curve="-180"/>
+<wire x1="137.16" y1="185.42" x2="137.16" y2="165.1" width="0.254" layer="103"/>
+<wire x1="137.16" y1="165.1" x2="132.08" y2="165.1" width="0.254" layer="103" curve="-180"/>
+<wire x1="187.96" y1="165.1" x2="99.06" y2="165.1" width="0.254" layer="102"/>
+<wire x1="99.06" y1="170.18" x2="187.96" y2="170.18" width="0.254" layer="105"/>
+<text x="141.478" y="170.942" size="2.54" layer="105" font="vector">0.75mm2</text>
+<text x="141.478" y="165.862" size="2.54" layer="102" font="vector">0.75mm2</text>
+</plain>
+<instances>
+<instance part="FRAME1" gate="G$1" x="0" y="0"/>
+<instance part="U$22" gate="G$1" x="228.6" y="175.26"/>
+<instance part="1/5" gate="PIN" x="187.96" y="185.42" rot="MR0"/>
+<instance part="1/6" gate="PIN" x="187.96" y="180.34" rot="MR0"/>
+<instance part="1/7" gate="PIN" x="187.96" y="170.18" rot="MR0"/>
+<instance part="1/8" gate="PIN" x="187.96" y="165.1" rot="MR0"/>
+<instance part="1/9" gate="PIN" x="99.06" y="185.42"/>
+<instance part="1/10" gate="PIN" x="99.06" y="180.34"/>
+<instance part="1/11" gate="PIN" x="99.06" y="170.18"/>
+<instance part="1/12" gate="PIN" x="99.06" y="165.1"/>
+<instance part="1/13" gate="G$1" x="68.58" y="175.26"/>
 </instances>
 <busses>
@@
 <dimension x1="190.5" y1="182.88" x2="182.88" y2="182.88" x3="175.26" y3="182.88" textsize="5.08" textratio="10" layer="103" dtype="leader" width="0.254"/>
 <dimension x1="124.46" y1="182.88" x2="182.88" y2="182.88" x3="175.26" y3="182.88" textsize="2.54" layer="103" dtype="leader" width="0.254"/>
-<text x="153.416" y="184.404" size="2.54" layer="103" font="vector">500mm</text>
+<text x="153.416" y="184.404" size="2.54" layer="103" font="vector">550mm</text>
 <wire x1="132.08" y1="172.72" x2="127" y2="172.72" width="0.254" layer="103" curve="-180"/>
 <wire x1="127" y1="177.8" x2="132.08" y2="177.8" width="0.254" layer="103" curve="-180"/>
@@
 <dimension x1="190.5" y1="165.1" x2="182.88" y2="165.1" x3="175.26" y3="165.1" textsize="5.08" textratio="10" layer="103" dtype="leader" width="0.254"/>
 <dimension x1="124.46" y1="165.1" x2="182.88" y2="165.1" x3="175.26" y3="165.1" textsize="2.54" layer="103" dtype="leader" width="0.254"/>
-<text x="153.416" y="166.624" size="2.54" layer="103" font="vector">500mm</text>
+<text x="153.416" y="166.624" size="2.54" layer="103" font="vector">600mm</text>
 <wire x1="132.08" y1="154.94" x2="127" y2="154.94" width="0.254" layer="103" curve="-180"/>
 <wire x1="127" y1="160.02" x2="132.08" y2="160.02" width="0.254" layer="103" curve="-180"/>
@@
 <dimension x1="337.82" y1="154.94" x2="330.2" y2="154.94" x3="322.58" y3="154.94" textsize="5.08" textratio="10" layer="103" dtype="leader" width="0.254"/>
 <dimension x1="271.78" y1="154.94" x2="330.2" y2="154.94" x3="322.58" y3="154.94" textsize="2.54" layer="103" dtype="leader" width="0.254"/>
-<text x="300.736" y="156.464" size="2.54" layer="103" font="vector">500mm</text>
+<text x="300.736" y="156.464" size="2.54" layer="103" font="vector">550mm</text>
 <wire x1="279.4" y1="144.78" x2="274.32" y2="144.78" width="0.254" layer="103" curve="-180"/>
 <wire x1="274.32" y1="149.86" x2="279.4" y2="149.86" width="0.254" layer="103" curve="-180"/>
@@
 <dimension x1="337.82" y1="137.16" x2="330.2" y2="137.16" x3="322.58" y3="137.16" textsize="5.08" textratio="10" layer="103" dtype="leader" width="0.254"/>
 <dimension x1="271.78" y1="137.16" x2="330.2" y2="137.16" x3="322.58" y3="137.16" textsize="2.54" layer="103" dtype="leader" width="0.254"/>
-<text x="300.736" y="138.684" size="2.54" layer="103" font="vector">500mm</text>
+<text x="300.736" y="138.684" size="2.54" layer="103" font="vector">600mm</text>
 <wire x1="279.4" y1="127" x2="274.32" y2="127" width="0.254" layer="103" curve="-180"/>
 <wire x1="274.32" y1="132.08" x2="279.4" y2="132.08" width="0.254" layer="103" curve="-180"/>
@@
 <dimension x1="190.5" y1="147.32" x2="182.88" y2="147.32" x3="175.26" y3="147.32" textsize="5.08" textratio="10" layer="103" dtype="leader" width="0.254"/>
 <dimension x1="124.46" y1="147.32" x2="182.88" y2="147.32" x3="175.26" y3="147.32" textsize="2.54" layer="103" dtype="leader" width="0.254"/>
-<text x="153.416" y="148.844" size="2.54" layer="103" font="vector">500mm</text>
+<text x="153.416" y="148.844" size="2.54" layer="103" font="vector">650mm</text>
 <wire x1="132.08" y1="137.16" x2="127" y2="137.16" width="0.254" layer="103" curve="-180"/>
 <wire x1="127" y1="142.24" x2="132.08" y2="142.24" width="0.254" layer="103" curve="-180"/>
@@
 <dimension x1="337.82" y1="119.38" x2="330.2" y2="119.38" x3="322.58" y3="119.38" textsize="5.08" textratio="10" layer="103" dtype="leader" width="0.254"/>
 <dimension x1="271.78" y1="119.38" x2="330.2" y2="119.38" x3="322.58" y3="119.38" textsize="2.54" layer="103" dtype="leader" width="0.254"/>
-<text x="300.736" y="120.904" size="2.54" layer="103" font="vector">500mm</text>
+<text x="300.736" y="120.904" size="2.54" layer="103" font="vector">650mm</text>
 <wire x1="279.4" y1="109.22" x2="274.32" y2="109.22" width="0.254" layer="103" curve="-180"/>
 <wire x1="274.32" y1="114.3" x2="279.4" y2="114.3" width="0.254" layer="103" curve="-180"/>
